File: ecad/_autosave-template.sch (KiCad schematic (older format))
At the start: 13 parts, among them P1 CF_EXP_LEFT, P2 CF_EXP_RIGHT, P3 CONN_2, P4 CONN_2, Q1 DMG2302U, Q2 DMG2302U

Commit message: modified schematic and pcb layout + plotted production files
Parts:
- P3, P4: footprint (none) -> Connector_Hirose:Hirose_DF13-02P-1.25DSA_1x02_P1.25mm_Vertical
Changed lines of the file:
@@
 F 0 "P3" H 5267 1637 40  0000 C CNN
 F 1 "CONN_2" H 5267 1713 40  0000 C CNN
-F 2 "" H 5400 1950 50  0001 C CNN
+F 2 "Connector_Hirose:Hirose_DF13-02P-1.25DSA_1x02_P1.25mm_Vertical" H 5400 1950 50  0001 C CNN
 F 3 "" H 5400 1950 50  0001 C CNN
 	1    5400 1950
@@
 F 0 "P4" H 8517 1637 40  0000 C CNN
 F 1 "CONN_2" H 8517 1713 40  0000 C CNN
-F 2 "" H 8650 1950 50  0001 C CNN
+F 2 "Connector_Hirose:Hirose_DF13-02P-1.25DSA_1x02_P1.25mm_Vertical" H 8650 1950 50  0001 C CNN
 F 3 "" H 8650 1950 50  0001 C CNN
 	1    8650 1950
-	-1   0    0    1
+	-1   0    0    -1
 $EndComp
 Wire Wire Line
